File: qfn-practice/qfn-practice.kicad_pcb (KiCad board)
At the start: 2 copper layers, 17.8 x 27.9 mm, 12 parts, among them J1 Conn_01x10, J2 Conn_01x10, J3 Conn_01x03, J4 Conn_01x04, J5 Conn_01x02, J7 Conn_01x03, U2 STM32F031G4Ux-thermal-pad

Commit message: small tweaks
Routing:
- net /ST_BOOT0: track 32.9 -> 33.5 mm

Commit message: add 2 layer gerbers
Parts:
- moved JP5 0.50 mm to (155.1, 74.1)
Routing:
- net /P11: track 28.8 -> 16.2 mm
- net GND: track 12.2 -> 10.4 mm, vias 23 -> 20
- added copper zone on In1.Cu, net GND
- added copper zone on In2.Cu, net GND
Other:
- copper layers 2 -> 4
- net class Default: clearance 0.15 -> 0.155
- rule trace_clearance: 0.15 -> 0.155

Commit message: 4 layer gerbers
Routing:
- net /ST_BOOT0: track 33.5 -> 15.7 mm, vias 0 -> 1
- net +3V3: track 48.3 -> 34.4 mm, vias 2 -> 4
- net GND: track 10.4 -> 24.0 mm, vias 20 -> 33
- net /ST_PA1: track 22.9 -> 17.3 mm
- net /P8: track 10.6 -> 8.40 mm
- net /P11: track 16.2 -> 17.5 mm
- net /AT_PB5_!RESET_ST_PF0: track 4.59 -> 5.71 mm
